File: cabane_minou/cabane_minou/cabane_minou.sch (KiCad schematic (older format))
At the start: 1 part

Commit message: Cabane minou Rev A0 envoyee
Parts:
- removed U?: 113990105, DIP2286W64P254L4826H735Q30N, symbol MCU_Module:113990105
- added C1, C2, C3: 100u, Capacitor_THT:CP_Radial_D8.0mm_P5.00mm, symbol Device:CP
- added D1: 1V, Diode_THT:D_A-405_P2.54mm_Vertical_AnodeUp, symbol Device:D_Zener
- added D2, D3, D4, D5: D_Schottky, Diode_THT:D_A-405_P2.54mm_Vertical_AnodeUp, symbol Device:D_Schottky
- added J1: Ext SPI, Connector_PinHeader_2.54mm:PinHeader_1x06_P2.54mm_Vertical, symbol Connector_Generic:Conn_01x06
- added J2: Lum, Connector_PinHeader_2.54mm:PinHeader_1x01_P2.54mm_Vertical, symbol Connector:Conn_01x01_Male
- added J3: Temp, Connector_PinHeader_2.54mm:PinHeader_1x01_P2.54mm_Vertical, symbol Connector:Conn_01x01_Male
- added J4: Bornier, TerminalBlock_Phoenix:TerminalBlock_Phoenix_MKDS-3-10-5.08_1x10_P5.08mm_Horizontal, symbol Connector_Generic:Conn_01x10
- added R1, R2: R, Resistor_THT:R_Axial_DIN0309_L9.0mm_D3.2mm_P2.54mm_Vertical, symbol Device:R
- added R10, R12, R7: 220, Resistor_THT:R_Axial_DIN0309_L9.0mm_D3.2mm_P2.54mm_Vertical, symbol Device:R
- added R11, R13, R14, R15, R3, R4, R5, R6, R8: 100k, Resistor_THT:R_Axial_DIN0309_L9.0mm_D3.2mm_P2.54mm_Vertical, symbol Device:R
- added R16, R9: 10, Resistor_THT:R_Axial_DIN0309_L9.0mm_D3.2mm_P2.54mm_Vertical, symbol Device:R
- added U1: NodeMCUs, bpc:BPC_NodeMCU_small, symbol bpc:NodeMCUs
Connections:
- new net: J2.1 (Pin_1), R1.2, U1.1 (A0_-_ADC_EX)
- new net: D2.2 (A), R3.2, R4.1, R9.2, U1.21 (D7_-_GPIO13_/_RXD2_/_HSPID)
- new net: R10.2, U1.22 (D6_-_GPIO12_/_HSPIQ)
- new net: J4.6 (Pin_6), R11.2, U1.23 (D5_-_GPIO14_/_HSPICLK)
- new net: R7.2, U1.26 (D4_-_GPIO2_/_TXD1)
- new net: R12.2, U1.28 (D2_-_GPIO4)
- new net: D4.2 (A), R13.2, R16.2, R5.2, U1.29 (D1_-_GPIO5)
- new net: D3.2 (A), J3.1 (Pin_1), J4.2 (Pin_2), R6.2, R8.1, U1.4 (D12_-_GPIO10_/_SD_D3)
- new net: D5.2 (A), J4.3 (Pin_3), R14.2, R15.1, U1.5 (D11_-_GPIO9_/_SD_D2)
- new net: J1.5 (Pin_5), U1.6 (SPI_INT_/_SD_D1)
- new net: J1.4 (Pin_4), U1.7 (SPI_MOSI_/_SD_CMD)
- new net: J1.3 (Pin_3), U1.8 (SPI_MISO_/_SD_D0)
- new net: J1.2 (Pin_2), U1.9 (SPI_CLK_/_SD_CLK)
- new net: D1.1 (K), R1.1, R2.2
- new net: J4.4 (Pin_4), R9.1
- new net: J4.5 (Pin_5), R10.1
- new net: J4.7 (Pin_7), R7.1
- new net: J4.8 (Pin_8), R12.1
- new net: J4.9 (Pin_9), R16.1
- new net +3V3: D2.1 (K), D3.1 (K), D4.1 (K), D5.1 (K), J1.6 (Pin_6), R11.1, R13.1, R14.1, R2.1, R3.1, R6.1, U1.11 (VDD3V3_1), U1.16 (VDD3V3_2), U1.25 (VDD3V3_3)
- new net +5V: C1.1, C2.1, C3.1, J4.10 (Pin_10), U1.15 (VDD5V)
- new net GND: C1.2, C2.2, C3.2, D1.2 (A), J1.1 (Pin_1), J4.1 (Pin_1), R15.2, R4.2, R5.1, R8.2, U1.10 (GND_1), U1.14 (GND_2), U1.17 (GND_3), U1.24 (GND_4)
- no-connect marks 0 -> 9
Other:
- note added: "1"
- note added: "28/03/2021"
- note added: "A0"
- note added: "CABANE DE MINOU (Bas/Tour/...)"
- note added: "Vers DHT Ext."
- note added: "Vers capteur lum."

Commit message: Réalisation du logiciel: - Webservice pour acces aux LEDs haut/bas de la cabane - Détection de mouvement et allumage: Vert pour haut, Rouge pour bas - Mise à jour du soft a distance
Correction schéma et PCB: Version B0:
- Trous de fixation (2.2 mm de diametre). Ils étaient un peu trop gros
- Simple diviseur pour l'entrée analogique: Non montées car déjà présentes sur NodeMcu
- ...
Parts:
- removed D1: 1V, Diode_THT:D_A-405_P2.54mm_Vertical_AnodeUp, symbol Device:D_Zener
- R1: value R -> 40k
- R2: value R -> 100k
Connections:
- net GND: now also R1.2
- net at J2.1 (Pin_1), U1.1 (A0_-_ADC_EX): now also R1.1, R2.2; no longer R1.2
Other:
- note added: "01/05/2021"
- note added: "B LD Bas"
- note added: "B LD Haut"
- note added: "B0"
- note added: "Capot"
- note added: "LED"
- note added: "Move Bas"
- note added: "Move Haut"
- note added: "Non"
- note added: "Non monté"
- note added: "Temp Bas"
- note added: "Temp Ext"
- note added: "monté"
- note removed: "28/03/2021"
- note removed: "A0"
Changed lines of the file:
@@
 U 1 1 6046DFE9
 P 3950 750
-F 0 "R2" H 4020 796 50  0000 L CNN
-F 1 "R" H 4020 705 50  0000 L CNN
+F 0 "R2" V 4100 600 50  0000 L CNN
+F 1 "100k" V 4100 800 50  0000 L CNN
 F 2 "Resistor_THT:R_Axial_DIN0309_L9.0mm_D3.2mm_P2.54mm_Vertical" V 3880 750 50  0001 C CNN
 F 3 "~" H 3950 750 50  0001 C CNN
@@
 	0    1    1    0
 $EndComp
-$Comp
-L Device:D_Zener D1
-U 1 1 60470D30
-P 3450 750
-F 0 "D1" V 3404 830 50  0000 L CNN
-F 1 "1V" V 3495 830 50  0000 L CNN
-F 2 "Diode_THT:D_A-405_P2.54mm_Vertical_AnodeUp" H 3450 750 50  0001 C CNN
-F 3 "~" H 3450 750 50  0001 C CNN
-	1    3450 750
-	-1   0    0    1
-$EndComp
 Wire Wire Line
 	3800 750  3750 750
@@
 Wire Wire Line
 	4250 750  4100 750
-$Comp
-L Device:R R1
-U 1 1 604719A0
-P 3450 1350
-F 0 "R1" V 3243 1350 50  0000 C CNN
-F 1 "R" V 3334 1350 50  0000 C CNN
-F 2 "Resistor_THT:R_Axial_DIN0309_L9.0mm_D3.2mm_P2.54mm_Vertical" V 3380 1350 50  0001 C CNN
-F 3 "~" H 3450 1350 50  0001 C CNN
-	1    3450 1350
-	0    1    1    0
-$EndComp
 Wire Wire Line
 	3750 1350 3750 750
@@
 U 1 1 604CDE74
 P 6900 3800
-F 0 "R6" H 6970 3846 50  0000 L CNN
-F 1 "100k" H 6970 3755 50  0000 L CNN
+F 0 "R6" H 6650 3900 50  0000 L CNN
+F 1 "100k" H 6650 3750 50  0000 L CNN
 F 2 "Resistor_THT:R_Axial_DIN0309_L9.0mm_D3.2mm_P2.54mm_Vertical" V 6830 3800 50  0001 C CNN
 F 3 "~" H 6900 3800 50  0001 C CNN
@@
 U 1 1 604CE110
 P 7200 3800
-F 0 "D3" V 7154 3880 50  0000 L CNN
-F 1 "D_Schottky" V 7245 3880 50  0000 L CNN
+F 0 "D3" V 7050 3850 50  0000 L CNN
+F 1 "D_Schottky" V 6950 3700 50  0000 L CNN
 F 2 "Diode_THT:D_A-405_P2.54mm_Vertical_AnodeUp" H 7200 3800 50  0001 C CNN
 F 3 "~" H 7200 3800 50  0001 C CNN
@@
 U 1 1 604D28C6
 P 7850 3800
-F 0 "R14" H 7920 3846 50  0000 L CNN
-F 1 "100k" H 7920 3755 50  0000 L CNN
+F 0 "R14" H 7600 3850 50  0000 L CNN
+F 1 "100k" H 7600 3700 50  0000 L CNN
 F 2 "Resistor_THT:R_Axial_DIN0309_L9.0mm_D3.2mm_P2.54mm_Vertical" V 7780 3800 50  0001 C CNN
 F 3 "~" H 7850 3800 50  0001 C CNN
@@
 U 1 1 604D2B98
 P 8150 3800
-F 0 "D5" V 8104 3880 50  0000 L CNN
-F 1 "D_Schottky" V 8195 3880 50  0000 L CNN
+F 0 "D5" V 8000 3850 50  0000 L CNN
+F 1 "D_Schottky" V 7900 3700 50  0000 L CNN
 F 2 "Diode_THT:D_A-405_P2.54mm_Vertical_AnodeUp" H 8150 3800 50  0001 C CNN
 F 3 "~" H 8150 3800 50  0001 C CNN
@@
 $EndComp
 Wire Wire Line
-	3750 1350 3600 1350
-Wire Wire Line
-	3300 1350 3200 1350
-Wire Wire Line
 	2950 1850 2950 1600
 Wire Wire Line
@@
 CABANE DE MINOU (Bas/Tour/...)
 Text Notes 8150 7650 0    50   ~ 0
-28/03/2021
+01/05/2021
 Text Notes 10600 7650 0    50   ~ 0
-A0
+B0
+Text Notes 9050 3400 1    50   ~ 0
+Temp Ext
+Text Notes 8750 3450 1    50   ~ 0
+Move Bas
+Text Notes 7900 3050 0    50   ~ 0
+Temp Bas
+Text Notes 7500 2650 0    50   ~ 0
+Capot
+Text Notes 7850 2750 0    50   ~ 0
+B LD Haut
+Text Notes 7900 2400 0    50   ~ 0
+LED
+Text Notes 7250 2200 0    50   ~ 0
+B LD Bas
+Text Notes 7500 1900 0    50   ~ 0
+Move Haut
+$Comp
+L Device:R R1
+U 1 1 608DF06D
+P 3450 750
+F 0 "R1" V 3600 650 50  0000 C CNN
+F 1 "40k" V 3600 850 50  0000 C CNN
+F 2 "Resistor_THT:R_Axial_DIN0309_L9.0mm_D3.2mm_P2.54mm_Vertical" V 3380 750 50  0001 C CNN
+F 3 "~" H 3450 750 50  0001 C CNN
+	1    3450 750
+	0    1    1    0
+$EndComp
+Wire Wire Line
+	3200 1350 3750 1350
+Wire Notes Line
+	3200 1100 4250 1100
+Wire Notes Line
+	4250 1100 4250 600
+Wire Notes Line
+	4250 600  3200 600
+Wire Notes Line
+	3200 600  3200 1100
+Text Notes 3800 1200 0    50   ~ 0
+Non monté
+Wire Notes Line
+	7350 4450 7350 4800
+Wire Notes Line
+	7350 4800 6800 4800
+Wire Notes Line
+	6800 4800 6800 4450
+Wire Notes Line
+	6800 4450 7350 4450
+Text Notes 6550 4900 0    50   ~ 0
+Non monté
+Wire Notes Line
+	6900 2800 6900 3100
+Wire Notes Line
+	6900 3100 6250 3100
+Wire Notes Line
+	6250 3100 6250 2800
+Wire Notes Line
+	6250 2800 6900 2800
+Text Notes 6300 2900 0    50   ~ 0
+Non
+Text Notes 6300 3000 0    50   ~ 0
+monté
+Wire Notes Line
+	8750 3700 8750 3900
+Wire Notes Line
+	8000 3900 8000 3700
+Text Notes 8300 3850 0    50   ~ 0
+Non monté
+Wire Notes Line
+	8000 3700 8750 3700
+Wire Notes Line
+	8000 3900 8750 3900
 $EndSCHEMATC
