File: cabane_minou/cabane_minou/cabane_minou.kicad_pcb (KiCad board)
At the start: 2 copper layers, 80 x 68 mm, 29 parts, among them J1 Ext SPI, J2 Lum, J3 Temp, J4 Bornier, U1 NodeMCUs

Commit message: Réalisation du logiciel: - Webservice pour acces aux LEDs haut/bas de la cabane - Détection de mouvement et allumage: Vert pour haut, Rouge pour bas - Mise à jour du soft a distance
Correction schéma et PCB: Version B0:
- Trous de fixation (2.2 mm de diametre). Ils étaient un peu trop gros
- Simple diviseur pour l'entrée analogique: Non montées car déjà présentes sur NodeMcu
- ...
Parts:
- removed D1: 1V, Diode_THT:D_A-405_P2.54mm_Vertical_AnodeUp
- R1: value R -> 40k
- R2: value R -> 100k
- moved R1 1.03 mm to (76.0, 93.0), turned to 180 degrees
Connections:
- R1 pad 1: Net-(D1-Pad1) -> Net-(J2-Pad1)
- R1 pad 2: Net-(J2-Pad1) -> GND
- R2 pad 2: Net-(D1-Pad1) -> Net-(J2-Pad1)
Routing:
- net Net-(J2-Pad1): track 10.2 -> 20.6 mm
- net Net-(D1-Pad1): track 9.27 -> 0.00 mm
Other:
- outline, holes or cut-outs redrawn
- board text added: "01/05/2021"
- board text added: "B0"
- board text added: "Rev B0"
- board text removed: "28/03/2021"
- board text removed: "A0"
- board text removed: "Rev A0"

Commit message: Nouvelle version de Cabane minou (Rev C)
Parts:
- added C10: 10µF, Capacitor_THT:CP_Radial_D4.0mm_P2.00mm, F.Cu at (143.5, 100.3)
- added C11: 10uF, Capacitor_THT:CP_Radial_D4.0mm_P2.00mm, B.Cu at (105.8, 109.1)
- added C12: 1n, Capacitor_THT:C_Disc_D5.0mm_W2.5mm_P2.50mm, F.Cu at (115.8, 109.1)
- added C13: 100nF, Capacitor_THT:C_Disc_D5.0mm_W2.5mm_P2.50mm, F.Cu at (56.0, 85.0)
- added C14: 10µF, Capacitor_THT:CP_Radial_D4.0mm_P2.00mm, F.Cu at (61.0, 97.0)
- added C16: 1n, Capacitor_THT:C_Disc_D5.0mm_W2.5mm_P2.50mm, B.Cu at (156.0, 80.5)
- added C18: 1n, Capacitor_THT:C_Disc_D5.0mm_W2.5mm_P2.50mm, B.Cu at (158.0, 62.5)
- added C19: 1n, Capacitor_THT:C_Disc_D5.0mm_W2.5mm_P2.50mm, F.Cu at (161.5, 92.0)
- added C20: 20uF, Capacitor_THT:CP_Radial_D8.0mm_P3.80mm, F.Cu at (152.5, 92.5)
- added C21: 100n, Capacitor_THT:C_Disc_D5.0mm_W2.5mm_P2.50mm, F.Cu at (115.0, 51.0)
- added C22: 100n, Capacitor_THT:C_Disc_D5.0mm_W2.5mm_P2.50mm, F.Cu at (84.5, 51.0)
- added C23: 100n, Capacitor_THT:C_Disc_D5.0mm_W2.5mm_P2.50mm, F.Cu at (184.7, 54.1)
- added C24: 100n, Capacitor_THT:C_Disc_D5.0mm_W2.5mm_P2.50mm, F.Cu at (164.3, 49.6)
- added C4: 100nF, Capacitor_THT:C_Disc_D5.0mm_W2.5mm_P2.50mm, F.Cu at (138.0, 79.5)
- added C5: 1n, Capacitor_THT:C_Disc_D5.0mm_W2.5mm_P2.50mm, F.Cu at (162.2, 129.9)
- added C6: 20uF, Capacitor_THT:CP_Radial_D8.0mm_P3.80mm, F.Cu at (170.2, 128.6)
- added C7: 10µF, Capacitor_THT:CP_Radial_D4.0mm_P2.00mm, F.Cu at (139.5, 88.5)
- added C8: 100n, Capacitor_THT:C_Disc_D5.0mm_W2.5mm_P2.50mm, F.Cu at (183.0, 105.5)
- added C9: 100nF, Capacitor_THT:C_Disc_D5.0mm_W2.5mm_P2.50mm, F.Cu at (131.5, 102.8)
- added D1: SR560, Diode_THT:D_DO-15_P12.70mm_Horizontal, F.Cu at (194.2, 138.5)
- added D10: DO-204, Diode_THT:D_A-405_P2.54mm_Vertical_AnodeUp, F.Cu at (136.5, 48.0)
- added D11: DO-204, Diode_THT:D_A-405_P2.54mm_Vertical_AnodeUp, F.Cu at (145.5, 51.0)
- added D12: DO-204, Diode_THT:D_A-405_P2.54mm_Vertical_AnodeUp, F.Cu at (77.7, 121.2)
- added D13: DO-204, Diode_THT:D_A-405_P2.54mm_Vertical_AnodeUp, F.Cu at (81.7, 123.3)
- added D14: DO-204, Diode_THT:D_A-405_P2.54mm_Vertical_AnodeUp, F.Cu at (188.2, 73.1)
- added D15: DO-204, Diode_THT:D_A-405_P2.54mm_Vertical_AnodeUp, F.Cu at (185.7, 77.1)
- added D16: DO-204, Diode_THT:D_A-405_P2.54mm_Vertical_AnodeUp, F.Cu at (187.7, 90.1)
- added D17: DO-204, Diode_THT:D_A-405_P2.54mm_Vertical_AnodeUp, F.Cu at (185.7, 86.1)
- added D6: DO-204, Diode_THT:D_A-405_P2.54mm_Vertical_AnodeUp, F.Cu at (95.7, 116.8)
- added D7: DO-204, Diode_THT:D_A-405_P2.54mm_Vertical_AnodeUp, F.Cu at (64.3, 50.8)
- added D8: DO-204, Diode_THT:D_A-405_P2.54mm_Vertical_AnodeUp, F.Cu at (64.3, 43.8)
- added D9: DO-201, Diode_THT:D_A-405_P2.54mm_Vertical_AnodeUp, F.Cu at (142.8, 126.7)
- added J10: Serial, TerminalBlock_Phoenix:TerminalBlock_Phoenix_MPT-0,5-4-2.54_1x04_P2.54mm_Horizontal, F.Cu at (199.0, 107.5)
- added J11: LEDs Res, TerminalBlock_Phoenix:TerminalBlock_Phoenix_MKDS-3-3-5.08_1x03_P5.08mm_Horizontal, F.Cu at (170.0, 34.0)
- added J12: Leds, Connector_JST:JST_EH_B3B-EH-A_1x03_P2.50mm_Vertical, F.Cu at (123.5, 127.7)
- added J13: Buttons, Connector_JST:JST_EH_B3B-EH-A_1x03_P2.50mm_Vertical, F.Cu at (54.0, 129.0)
- added J14: Couvercle, Connector_JST:JST_EH_B6B-EH-A_1x06_P2.50mm_Vertical, F.Cu at (59.0, 49.5)
- added J15: Commande 12V, TerminalBlock_Phoenix:TerminalBlock_Phoenix_MKDS-1,5-2-5.08_1x02_P5.08mm_Horizontal, F.Cu at (147.7, 134.2)
- added J5: LEDs Bas, TerminalBlock_Phoenix:TerminalBlock_Phoenix_MKDS-3-3-5.08_1x03_P5.08mm_Horizontal, F.Cu at (90.1, 34.0)
- added J6: Move Tour, TerminalBlock_Phoenix:TerminalBlock_Phoenix_MKDS-3-4-5.08_1x04_P5.08mm_Horizontal, F.Cu at (201.7, 89.1)
- added J7: LEDs Tour, TerminalBlock_Phoenix:TerminalBlock_Phoenix_MKDS-3-3-5.08_1x03_P5.08mm_Horizontal, F.Cu at (202.0, 60.1)
- added J8: Move Haut, TerminalBlock_Phoenix:TerminalBlock_Phoenix_MKDS-3-3-5.08_1x03_P5.08mm_Horizontal, F.Cu at (149.0, 34.0)
- added J9: LEDs Haut, TerminalBlock_Phoenix:TerminalBlock_Phoenix_MKDS-3-3-5.08_1x03_P5.08mm_Horizontal, F.Cu at (121.0, 34.0)
- added Q1: BPC_2N2222A, Package_TO_SOT_THT:TO-92, F.Cu at (137.9, 70.5)
- added Q10: BC327, Package_TO_SOT_THT:TO-92_Inline, F.Cu at (90.0, 43.0)
- added Q11: BPC_2N2222A, Package_TO_SOT_THT:TO-92, F.Cu at (190.4, 55.3)
- added Q12: BPC_2N2222A, Package_TO_SOT_THT:TO-92, F.Cu at (166.1, 44.9)
- added Q13: BC327, Package_TO_SOT_THT:TO-92_Inline, F.Cu at (193.2, 60.1)
- added Q14: BC327, Package_TO_SOT_THT:TO-92_Inline, F.Cu at (170.8, 42.3)
- added Q2: BC327, Package_TO_SOT_THT:TO-92_Inline, F.Cu at (137.9, 75.5)
- added Q3: BPC_2N2222A, Package_TO_SOT_THT:TO-92, F.Cu at (188.0, 108.0)
- added Q4: BC327, Package_TO_SOT_THT:TO-92_Inline, F.Cu at (193.0, 108.0)
- added Q5: BPC_2N2222A, Package_TO_SOT_THT:TO-92, F.Cu at (151.8, 118.2)
- added Q6: BPC_IPP034N03L, Package_TO_SOT_THT:TO-220-3_Vertical, F.Cu at (152.9, 122.2)
- added Q7: BPC_2N2222A, Package_TO_SOT_THT:TO-92, F.Cu at (116.0, 45.3)
- added Q8: BPC_2N2222A, Package_TO_SOT_THT:TO-92, F.Cu at (85.0, 45.5)
- added Q9: BC327, Package_TO_SOT_THT:TO-92_Inline, F.Cu at (121.0, 42.7)
- added R17: 100k, Resistor_THT:R_Axial_DIN0204_L3.6mm_D1.6mm_P7.62mm_Horizontal, F.Cu at (59.8, 125.0)
- added R18: 220, Resistor_THT:R_Axial_DIN0204_L3.6mm_D1.6mm_P7.62mm_Horizontal, F.Cu at (55.3, 39.2)
- added R19: 100k, Resistor_THT:R_Axial_DIN0204_L3.6mm_D1.6mm_P7.62mm_Horizontal, F.Cu at (59.8, 133.0)
- added R20: 220, Resistor_THT:R_Axial_DIN0204_L3.6mm_D1.6mm_P7.62mm_Horizontal, F.Cu at (141.0, 116.2)
- added R21: 100k, Resistor_THT:R_Axial_DIN0204_L3.6mm_D1.6mm_P7.62mm_Horizontal, F.Cu at (141.0, 119.2)
- added R22: 10, Resistor_THT:R_Axial_DIN0204_L3.6mm_D1.6mm_P7.62mm_Horizontal, F.Cu at (91.7, 116.3)
- added R23: 10, Resistor_THT:R_Axial_DIN0204_L3.6mm_D1.6mm_P7.62mm_Horizontal, F.Cu at (49.3, 42.2)
- added R24: 100k, Resistor_THT:R_Axial_DIN0204_L3.6mm_D1.6mm_P7.62mm_Horizontal, F.Cu at (147.0, 127.2)
- added R25: 1k, Resistor_THT:R_Axial_DIN0204_L3.6mm_D1.6mm_P7.62mm_Horizontal, F.Cu at (98.7, 123.9)
- added R26: 100k, Resistor_THT:R_Axial_DIN0204_L3.6mm_D1.6mm_P7.62mm_Horizontal, F.Cu at (52.3, 49.9)
- added R27: 100k, Resistor_THT:R_Axial_DIN0204_L3.6mm_D1.6mm_P7.62mm_Horizontal, F.Cu at (107.7, 124.1)
- added R28: 10, Resistor_THT:R_Axial_DIN0204_L3.6mm_D1.6mm_P7.62mm_Horizontal, F.Cu at (150.8, 42.0)
- added R29: 10, Resistor_THT:R_Axial_DIN0204_L3.6mm_D1.6mm_P7.62mm_Horizontal, F.Cu at (87.7, 124.1)
- added R30: 10, Resistor_THT:R_Axial_DIN0204_L3.6mm_D1.6mm_P7.62mm_Horizontal, F.Cu at (184.9, 80.1)
- added R31: 10, Resistor_THT:R_Axial_DIN0204_L3.6mm_D1.6mm_P7.62mm_Horizontal, F.Cu at (184.9, 83.1)
- added R32: 100k, Resistor_THT:R_Axial_DIN0204_L3.6mm_D1.6mm_P7.62mm_Horizontal, F.Cu at (136.2, 45.0)
- added R33: 100k, Resistor_THT:R_Axial_DIN0204_L3.6mm_D1.6mm_P7.62mm_Horizontal, F.Cu at (143.2, 48.0)
- added R34: 100k, Resistor_THT:R_Axial_DIN0204_L3.6mm_D1.6mm_P7.62mm_Horizontal, F.Cu at (77.7, 118.6)
- added R35: 100k, Resistor_THT:R_Axial_DIN0204_L3.6mm_D1.6mm_P7.62mm_Horizontal, F.Cu at (81.7, 111.0)
- added R36: 100k, Resistor_THT:R_Axial_DIN0204_L3.6mm_D1.6mm_P7.62mm_Horizontal, F.Cu at (178.5, 72.3)
- added R37: 100k, Resistor_THT:R_Axial_DIN0204_L3.6mm_D1.6mm_P7.62mm_Horizontal, F.Cu at (178.7, 82.1)
- added R38: 100k, Resistor_THT:R_Axial_DIN0204_L3.6mm_D1.6mm_P7.62mm_Horizontal, F.Cu at (173.7, 72.3)
- added R39: 100k, Resistor_THT:R_Axial_DIN0204_L3.6mm_D1.6mm_P7.62mm_Horizontal, F.Cu at (173.7, 82.1)
- added R40: 220, Resistor_THT:R_Axial_DIN0204_L3.6mm_D1.6mm_P7.62mm_Horizontal, F.Cu at (109.0, 49.8)
- added R41: 220, Resistor_THT:R_Axial_DIN0204_L3.6mm_D1.6mm_P7.62mm_Horizontal, F.Cu at (78.0, 49.8)
- added R42: 100k, Resistor_THT:R_Axial_DIN0204_L3.6mm_D1.6mm_P7.62mm_Horizontal, F.Cu at (114.2, 54.0)
- added R43: 100k, Resistor_THT:R_Axial_DIN0204_L3.6mm_D1.6mm_P7.62mm_Horizontal, F.Cu at (84.0, 54.0)
- added R44: 100k, Resistor_THT:R_Axial_DIN0204_L3.6mm_D1.6mm_P7.62mm_Horizontal, F.Cu at (126.0, 46.6)
- added R45: 100k, Resistor_THT:R_Axial_DIN0204_L3.6mm_D1.6mm_P7.62mm_Horizontal, F.Cu at (95.0, 46.6)
- added R46: 50, Resistor_THT:R_Axial_DIN0204_L3.6mm_D1.6mm_P7.62mm_Horizontal, F.Cu at (81.0, 49.8)
- added R47: 50, Resistor_THT:R_Axial_DIN0204_L3.6mm_D1.6mm_P7.62mm_Horizontal, F.Cu at (112.0, 49.8)
- added R48: 50, Resistor_THT:R_Axial_DIN0204_L3.6mm_D1.6mm_P7.62mm_Horizontal, F.Cu at (185.9, 51.1)
- added R49: 50, Resistor_THT:R_Axial_DIN0204_L3.6mm_D1.6mm_P7.62mm_Horizontal, F.Cu at (160.8, 49.4)
- added R50: 220, Resistor_THT:R_Axial_DIN0204_L3.6mm_D1.6mm_P7.62mm_Horizontal, F.Cu at (185.9, 48.1)
- added R51: 220, Resistor_THT:R_Axial_DIN0204_L3.6mm_D1.6mm_P7.62mm_Horizontal, F.Cu at (157.8, 49.4)
- added R52: 100k, Resistor_THT:R_Axial_DIN0204_L3.6mm_D1.6mm_P7.62mm_Horizontal, F.Cu at (181.7, 54.3)
- added R53: 100k, Resistor_THT:R_Axial_DIN0204_L3.6mm_D1.6mm_P7.62mm_Horizontal, F.Cu at (164.0, 52.6)
- added R54: 100k, Resistor_THT:R_Axial_DIN0204_L3.6mm_D1.6mm_P7.62mm_Horizontal, F.Cu at (189.9, 65.1)
- added R55: 100k, Resistor_THT:R_Axial_DIN0204_L3.6mm_D1.6mm_P7.62mm_Horizontal, F.Cu at (174.8, 45.4)
- added TH1: Thermistor_NTC, Resistor_THT:R_Axial_DIN0204_L3.6mm_D1.6mm_P7.62mm_Horizontal, F.Cu at (190.2, 133.5)
- added U2: LM1117DT-3.3, Package_TO_SOT_THT:TO-220-3_Vertical, F.Cu at (142.0, 82.6)
- added U3: BPC_ATMEGA2560_PRO, bpc:BPC_ATMEGA2560_PRO_MINI, F.Cu at (95.0, 89.0)
- added U4: ~, bpc:BPC_HC05_Vertical, F.Cu at (124.0, 82.0)
- added U5: RtcArduino, bpc:BPC_RtcArduino, B.Cu at (52.0, 76.0)
- added U6: BPC_ESP8266-01_ESP-01, bpc:BPC_XCVR_ESP8266-01_ESP-01, F.Cu at (157.3, 77.2)
- added U7: ~, bpc:BPC_LVLCONV_5_33, B.Cu at (163.2, 77.0)
- added X1: Trou, bpc:BPC_Trou4mm_Fixation, F.Cu at (210.0, 139.0)
- added X2: Trou, bpc:BPC_Trou4mm_Fixation, F.Cu at (42.0, 139.0)
- added X3: Trou, bpc:BPC_Trou4mm_Fixation, F.Cu at (210.0, 27.0)
- added X4: Trou, bpc:BPC_Trou4mm_Fixation, F.Cu at (42.0, 27.0)
- C1, C3: value 100u -> 100n; footprint Capacitor_THT:CP_Radial_D8.0mm_P5.00mm -> Capacitor_THT:C_Disc_D5.0mm_W2.5mm_P2.50mm
- C2: value 100u -> 40uF; footprint Capacitor_THT:CP_Radial_D8.0mm_P5.00mm -> Capacitor_THT:CP_Radial_D8.0mm_P3.80mm
- D2, D3, D5: value D_Schottky -> DO-204
- D4: value D_Schottky -> D; moved to B.Cu
- J1: value Ext SPI -> Alim 12V; footprint Connector_PinHeader_2.54mm:PinHeader_1x06_P2.54mm_Vertical -> TerminalBlock_Phoenix:TerminalBlock_Phoenix_MKDS-1,5-2-5.08_1x02_P5.08mm_Horizontal
- J2: value Lum -> Log; footprint Connector_PinHeader_2.54mm:PinHeader_1x01_P2.54mm_Vertical -> Connector_JST:JST_XH_B4B-XH-AM_1x04_P2.50mm_Vertical
- J3: value Temp -> Screen; footprint Connector_PinHeader_2.54mm:PinHeader_1x01_P2.54mm_Vertical -> Connector_JST:JST_XH_B4B-XH-A_1x04_P2.50mm_Vertical
- J4: value Bornier -> Bas; footprint TerminalBlock_Phoenix:TerminalBlock_Phoenix_MKDS-3-10-5.08_1x10_P5.08mm_Horizontal -> TerminalBlock_Phoenix:TerminalBlock_Phoenix_MKDS-3-6-5.08_1x06_P5.08mm_Horizontal
- R1: value 40k -> 220; footprint Resistor_THT:R_Axial_DIN0309_L9.0mm_D3.2mm_P2.54mm_Vertical -> Resistor_THT:R_Axial_DIN0204_L3.6mm_D1.6mm_P7.62mm_Horizontal
- R10: value 220 -> 100; footprint Resistor_THT:R_Axial_DIN0309_L9.0mm_D3.2mm_P2.54mm_Vertical -> Resistor_THT:R_Axial_DIN0204_L3.6mm_D1.6mm_P7.62mm_Horizontal
- R11: value 100k -> 10k; footprint Resistor_THT:R_Axial_DIN0309_L9.0mm_D3.2mm_P2.54mm_Vertical -> Resistor_THT:R_Axial_DIN0204_L3.6mm_D1.6mm_P7.62mm_Horizontal; moved to B.Cu
- R12: value 220 -> 10k; footprint Resistor_THT:R_Axial_DIN0309_L9.0mm_D3.2mm_P2.54mm_Vertical -> Resistor_THT:R_Axial_DIN0204_L3.6mm_D1.6mm_P7.62mm_Horizontal; moved to B.Cu
- R13, R15, R6: value 100k -> 220; footprint Resistor_THT:R_Axial_DIN0309_L9.0mm_D3.2mm_P2.54mm_Vertical -> Resistor_THT:R_Axial_DIN0204_L3.6mm_D1.6mm_P7.62mm_Horizontal
- R14, R2, R3, R4, R8: footprint Resistor_THT:R_Axial_DIN0309_L9.0mm_D3.2mm_P2.54mm_Vertical -> Resistor_THT:R_Axial_DIN0204_L3.6mm_D1.6mm_P7.62mm_Horizontal
- R16: value 10 -> 220; footprint Resistor_THT:R_Axial_DIN0309_L9.0mm_D3.2mm_P2.54mm_Vertical -> Resistor_THT:R_Axial_DIN0204_L3.6mm_D1.6mm_P7.62mm_Horizontal
- R5: value 100k -> 30k; footprint Resistor_THT:R_Axial_DIN0309_L9.0mm_D3.2mm_P2.54mm_Vertical -> Resistor_THT:R_Axial_DIN0204_L3.6mm_D1.6mm_P7.62mm_Horizontal
- R7: value 220 -> 100k; footprint Resistor_THT:R_Axial_DIN0309_L9.0mm_D3.2mm_P2.54mm_Vertical -> Resistor_THT:R_Axial_DIN0204_L3.6mm_D1.6mm_P7.62mm_Horizontal
- R9: value 10 -> 100; footprint Resistor_THT:R_Axial_DIN0309_L9.0mm_D3.2mm_P2.54mm_Vertical -> Resistor_THT:R_Axial_DIN0204_L3.6mm_D1.6mm_P7.62mm_Horizontal
- U1: value NodeMCUs -> BPC_Alim5V; footprint bpc:BPC_NodeMCU_small -> bpc:BPC_Alim5V; moved to B.Cu
- moved J1 129.6 mm to (202.5, 125.2), turned to 90 degrees
- moved C3 114.0 mm to (187.2, 129.4), turned to -90 degrees
- moved R14 97.0 mm to (55.3, 49.9), turned to 90 degrees
- moved U1 91.6 mm to (184.2, 123.9), turned to 180 degrees
- moved J3 74.1 mm to (55.5, 90.0), turned to 0 degrees
- moved R1 73.2 mm to (144.3, 66.5)
- moved R5 70.5 mm to (176.3, 120.7), turned to 0 degrees
- moved R8 70.0 mm to (193.8, 102.5)
- moved R2 67.2 mm to (134.5, 68.7), turned to -90 degrees
- moved R12 66.7 mm to (49.7, 73.0), turned to 0 degrees
- moved R7 65.8 mm to (177.0, 100.8), turned to -90 degrees
- moved C2 65.5 mm to (179.2, 128.6), turned to -90 degrees
- moved J2 62.1 mm to (136.5, 105.8), turned to 90 degrees
- moved J4 61.1 mm to (80.3, 132.3), turned to 0 degrees
- moved R6 59.0 mm to (180.0, 108.5), turned to 90 degrees
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Connections:
- C1 pad 1: +5V -> Net-(C1-Pad1)
- C2 pad 1: +5V -> 12V
- C3 pad 1: +5V -> 12V
- D2 pad 1: +3V3 -> +5V
- D2 pad 2: Net-(D2-Pad2) -> UC_IN_MES_12V
- D3 pad 1: +3V3 -> UC_IN_MES_12V
- D3 pad 2: Net-(D3-Pad2) -> GND
- D4 pad 1: +3V3 -> Net-(D4-K)
- D4 pad 2: Net-(D4-Pad2) -> +5V
- D5 pad 1: +3V3 -> +5V
- D5 pad 2: Net-(D5-Pad2) -> UC_IN_CAPOT
- J1 pad 1: GND -> Net-(D1-A)
- J1 pad 2: Net-(J1-Pad2) -> GND
- J2 pad 1: Net-(J2-Pad1) -> +5V
- J3 pad 1: Net-(D3-Pad2) -> +5V
- J4 pad 1: GND -> +5V
- J4 pad 2: Net-(D3-Pad2) -> OUT_LED_CAPOT_OUVERT
- J4 pad 3: Net-(D5-Pad2) -> IN_CAPOT
- J4 pad 4: Net-(J4-Pad4) -> TEMP_BAS
- J4 pad 5: Net-(J4-Pad5) -> IN_PRESENCE_BAS
- J4 pad 6: Net-(J4-Pad6) -> GND
- R1 pad 1: Net-(J2-Pad1) -> UC_3V_ESP
- R1 pad 2: GND -> Net-(C1-Pad1)
- R10 pad 1: Net-(J4-Pad5) -> Net-(U4-RXD)
- R10 pad 2: Net-(R10-Pad2) -> UC_TX_PROG
- R11 pad 1: +3V3 -> +5V
- R11 pad 2: Net-(J4-Pad6) -> SCL
- R12 pad 1: Net-(J4-Pad8) -> +5V
- R12 pad 2: Net-(R12-Pad2) -> SDA
- R13 pad 1: +3V3 -> OUT_LED_CAPOT_OUVERT
- R13 pad 2: Net-(D4-Pad2) -> UC_OUT_LED_CAPOT_OUVERT
- R14 pad 1: +3V3 -> +5V
- R14 pad 2: Net-(D5-Pad2) -> UC_IN_SW1_BUTTON
- R15 pad 1: Net-(D5-Pad2) -> Net-(J12-Pin_1)
- R15 pad 2: GND -> UC_OUT_LED_2
- R16 pad 1: Net-(J4-Pad9) -> Net-(J12-Pin_2)
- R16 pad 2: Net-(D4-Pad2) -> UC_OUT_LED_3
- R2 pad 1: +3V3 -> Net-(C1-Pad1)
- R2 pad 2: Net-(J2-Pad1) -> GND
- R3 pad 1: +3V3 -> +5V
- R3 pad 2: Net-(D2-Pad2) -> Net-(Q2-B)
- R4 pad 1: Net-(D2-Pad2) -> 12V
- R4 pad 2: GND -> UC_IN_MES_12V
- R5 pad 1: GND -> UC_IN_MES_12V
- R5 pad 2: Net-(D4-Pad2) -> GND
- R6 pad 1: +3V3 -> UC_5V_SER
- R6 pad 2: Net-(D3-Pad2) -> Net-(C8-Pad1)
- R7 pad 1: Net-(J4-Pad7) -> Net-(C8-Pad1)
- R7 pad 2: Net-(R7-Pad2) -> GND
- R8 pad 1: Net-(D3-Pad2) -> +5V
- R8 pad 2: GND -> Net-(Q4-B)
- R9 pad 1: Net-(J4-Pad4) -> UC_RX_PROG
- R9 pad 2: Net-(D2-Pad2) -> Net-(U4-TXD)
- U1 pad 1: Net-(J2-Pad1) -> 12V
- U1 pad 2: Net-(U1-Pad2) -> 12V
- U1 pad 3: Net-(U1-Pad3) -> GND
- U1 pad 4: Net-(D3-Pad2) -> GND
- U1 pad 5: Net-(D5-Pad2) -> GND
- U1 pad 6: Net-(J1-Pad5) -> GND
- U1 pad 7: Net-(J1-Pad4) -> +5V
- U1 pad 8: Net-(J1-Pad3) -> +5V
Routing:
- net +5V: track 121.6 -> 333.7 mm
- net +3V3: track 202.2 -> 0.00 mm, vias 4 -> 0
- net Net-(D5-Pad2): track 117.4 -> 0.00 mm, vias 2 -> 0
- net Net-(D3-Pad2): track 106.2 -> 0.00 mm, vias 1 -> 0
- net UC_IN_PRESENCE_HAUT: track 0.00 -> 87.2 mm
- net UC_OUT_LEDS_RES: track 0.00 -> 79.1 mm
- net UC_5V_LEDS_RES: track 0.00 -> 77.6 mm
- net POWER_12V: track 0.00 -> 72.6 mm
- net UC_5V_LEDS_TOUR: track 0.00 -> 68.1 mm
- net UC_OUT_LEDS_TOUR: track 0.00 -> 67.2 mm
- net Net-(J4-Pad6): track 44.0 -> 0.00 mm, vias 1 -> 0
- net UC_5V_LEDS_HAUT: track 0.00 -> 41.1 mm
- net 12V: track 0.00 -> 40.2 mm, vias 0 -> 1
- net UC_OUT_LEDS_HAUT: track 0.00 -> 39.8 mm
- net POWER_3.3: track 0.00 -> 39.8 mm
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- removed copper zone on B.Cu, net GND
- removed copper zone on F.Cu, net GND
Other:
- board size 80 x 68 mm -> 176 x 120 mm
- net class 3.3V removed
- net class 5V removed
- net class Default removed
- net class GND removed
- board text removed: "(BPC 2021)"
- board text removed: "01/05/2021"
- board text removed: "1/1"
- board text removed: "B0"
- board text removed: "By Poloisirs"
- board text removed: "CABANE DE MINOU (Bas/Tour/...)"
- board text removed: "Cabane Minou"
- board text removed: "Rev B0"
