File: cabane_minou/cabane_minou/cpu.kicad_sch (KiCad schematic)
At the start: 26 parts, among them J2 Log, J3 Screen, U3 BPC_ATMEGA2560_PRO

Commit message: Design cabane minou "version 2024"
Parts:
- added C?: 1n, Capacitor_THT:C_Disc_D5.0mm_W2.5mm_P2.50mm, symbol Device:C
- added C?: 10uF, Capacitor_THT:CP_Radial_D4.0mm_P2.00mm, symbol Device:C_Polarized
- D?: footprint Diode_THT:D_A-405_P2.54mm_Vertical_AnodeUp -> Diode_THT:D_5W_P12.70mm_Horizontal
- J2: footprint Connector_JST:JST_XH_B4B-XH-AM_1x04_P2.50mm_Vertical -> Connector_JST:JST_XH_B4B-XH-A_1x04_P2.50mm_Vertical
Connections:
- net GND: now also C?.2, C?.2
- net LUMINOSITE: now also U3.A14; no longer U3.A1
- net UC_3V_ESP: now also U3.D41; no longer U3.D9
- net UC_5V_LEDS_BAS: now also U3.D30; no longer U3.D26
- net UC_5V_LEDS_HAUT: now also U3.D28; no longer U3.D30
- net UC_5V_LEDS_RES: now also U3.D26; no longer U3.D27
- net UC_5V_LEDS_TOUR: now also U3.D22; no longer U3.D23
- net UC_5V_SER: now also U3.D24; no longer U3.D35
- net UC_IN_CAPOT: now also U3.D32; no longer U3.D41
- net UC_IN_MES_12V: now also U3.A15; no longer U3.A0
- net UC_IN_PRESENCE_BAS: now also U3.D36; no longer U3.D38
- net UC_IN_PRESENCE_HAUT: now also U3.D27; no longer U3.D29
- net UC_IN_PRESENCE_TOUR_BAS: now also U3.D37
- net UC_IN_PRESENCE_TOUR_HAUT: now also U3.D39
- net UC_IN_SW1_BUTTON: now also U3.D40; no longer U3.D3
- net UC_IN_SW2_BUTTON: now also U3.D3; no longer U3.D5
- net UC_IN_SW3_BUTTON: now also U3.D5; no longer U3.D7
- net UC_IO1: now also U3.D7; no longer U3.D22
- net UC_IO2: now also U3.D9; no longer U3.D24
- net UC_OUT_CMD_CHAUFFAGE: now also U3.D2; no longer U3.D45
- net UC_OUT_LEDS_BAS: now also U3.D31; no longer U3.D28
- net UC_OUT_LEDS_HAUT: now also U3.D29; no longer U3.D31
- net UC_OUT_LEDS_TOUR: now also U3.D23
- net UC_OUT_LED_1: now also U3.D43; no longer U3.D2
- net UC_OUT_LED_CAPOT_OUVERT: now also U3.D34; no longer U3.D40
- net UC_TEMP_BAS: now also U3.D38; no longer U3.D43
- net at C?.1, C?.1, D?.1 (K)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: now also C?.1, C?.1
- no-connect marks 45 -> 47
Other:
- note added: "1 cmd Alim module croquettes 1 cmd moteur croquettes 1 cmd vibreur croquettes 1 detecteur croquettes vides 1 cmd pompe eau fontaine 1 cmd LED fontaine"
