File: cabane_minou/cabane_minou/power.kicad_sch (KiCad schematic)
At the start: 27 parts, among them Q1 BPC_2N2222A, Q2 BC327, Q3 BPC_2N2222A, Q4 BC327, U2 LM1117DT-3.3

Commit message: Amélioration design du PCB (contour) Adaptation à la boîte Ajout datasheets
Changed lines of the file:
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@@
   (title_block
     (title "Cabane à Minou")
-    (rev "B0")
+    (date "2024-11-27")
+    (rev "Rev C0")
     (company "BPC")
-    (comment 1 "2 capteurs de température / 3 entrées détecteur de mouvement")
-    (comment 2 "Wifi / Luminosité / RTC")
+    (comment 1 "2 capteurs de température / 4 entrées détecteur de mouvement")
+    (comment 2 "Wifi / Luminosité / RTC / Bluetooth / Lcd")
     (comment 3 "4 sorties Strip LEDs (Avec Alim. 5V pilotable)")
     (comment 4 "Alimentation 12V / 1 sortie 12V commutable")
@@
   (junction (at 50.8 25.4) (diameter 0) (color 0 0 0 0)
   )
+  (junction (at 71.12 25.4) (diameter 0) (color 0 0 0 0)
+  )
   (junction (at 62.23 25.4) (diameter 0) (color 0 0 0 0)
   )
@@
     (stroke (width 0) (type default))
   )
-  (wire (pts (xy 68.58 25.4) (xy 73.66 25.4))
+  (wire (pts (xy 68.58 25.4) (xy 71.12 25.4))
     (stroke (width 0) (type default))
   )
@@
     (stroke (width 0) (type default))
   )
+  (wire (pts (xy 71.12 22.86) (xy 71.12 25.4))
+    (stroke (width 0) (type default))
+  )
   (wire (pts (xy 226.06 132.08) (xy 226.06 137.16))
     (stroke (width 0) (type default))
@@
   )
   (wire (pts (xy 58.42 129.54) (xy 58.42 132.08))
+    (stroke (width 0) (type default))
+  )
+  (wire (pts (xy 71.12 25.4) (xy 73.66 25.4))
     (stroke (width 0) (type default))
   )
@@
         )
       )
+    )
+  )
+  (symbol (lib_id "power:PWR_FLAG") (at 71.12 22.86 0) (unit 1)
+    (in_bom yes) (on_board yes) (dnp no) (fields_autoplaced)
+    (property "Reference" "#FLG04" (at 71.12 20.955 0)
+      (effects (font (size 1.27 1.27)) hide)
+    )
+    (property "Value" "PWR_FLAG" (at 71.12 18.915 0)
+      (effects (font (size 1.27 1.27)))
+    )
+    (property "Footprint" "" (at 71.12 22.86 0)
+      (effects (font (size 1.27 1.27)) hide)
+    )
+    (property "Datasheet" "~" (at 71.12 22.86 0)
+      (effects (font (size 1.27 1.27)) hide)
+    )
+    (pin "1")
+    (instances
+      (project "cabane_minou"
+        (path "/11e62a2f-8df1-4cb5-ab57-f2733cc2df79/5dbc7775-50ea-4fbb-95fe-87fffe8eb81e"
+          (reference "#FLG04") (unit 1)
+        )
+      )
