File: cabane_minou/hard/power.kicad_sch (KiCad schematic)
At the start: 27 parts, among them Q1 BPC_2N2222A, Q2 BC327, Q3 BPC_2N2222A, Q4 BC327, U2 LM1117DT-3.3

Commit message: Renommage dossier hard Création nouvelle version de soft (pour la nouvelle carte 2024)
Other:
- note added: "Erreur Q6: Pas la bonne empreinte MOS Nau lieu d'un P !!!!! TH1 pas assez large + trous trops fins D9 et D4 trop grands + trous trops gros Empreintes de R22, R23, R28, R29, R30 et R31 de 10 Ohms trop petites au moins 10mm Modifier J14 pour être de même type que les autres Mettre 100 nF sur Q5 comme pour les autres Mettre une pullup de 10k sur les entrées temp (avant la 10R cote DHT)"
Changed lines of the file:
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@@
     (stroke (width 0) (type default))
+  )
+  (text "Erreur Q6: Pas la bonne empreinte MOS Nau lieu d'un P !!!!!\nTH1 pas assez large + trous trops fins\nD9 et D4 trop grands + trous trops gros\nEmpreintes de R22, R23, R28, R29, R30 et R31 de 10 Ohms trop petites au moins 10mm \nModifier J14 pour être de même type que les autres\nMettre 100 nF sur Q5 comme pour les autres\nMettre une pullup de 10k sur les entrées temp (avant la 10R cote DHT)\n"
+    (at 90.17 162.56 0)
+    (effects (font (size 1.27 1.27)) (justify left bottom))
   )
   (text "Verif pinout micro = schéma = empreinte\nVerif EN du buffer et aussi son empreinte"
