File: cabane_minou/hard/es.kicad_sch (KiCad schematic)
At the start: 54 parts, among them J10 Serial, J11 LEDs Res, J12 Leds, J13 Buttons, J14 Couvercle, J5 LEDs Bas, J6 Move Tour, J7 LEDs Tour, J8 Move Haut, J9 LEDs Haut

Commit message: Début corrections suite utilisation en 2025...
Parts:
- Q?: value BPC_IPP034N03L -> P03P4L-04; symbol bpc:BPC_IPP034N03L -> bpc:P03P4L-04
Connections:
- net POWER_12V: now also Q?.3 (S); no longer Q?.2 (D)
- net at D?.2 (A), J?.1 (Pin_1): now also Q?.2 (D); no longer Q?.3 (S)
Changed lines of the file:
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@@
     )
   )
-  (symbol (lib_id "bpc:BPC_IPP034N03L") (at 158.75 46.99 0) (unit 1)
+  (symbol (lib_id "bpc:P03P4L-04") (at 158.75 46.99 0) (unit 1)
     (in_bom yes) (on_board yes) (dnp no) (fields_autoplaced)
-    (property "Reference" "Q?" (at 163.957 45.966 0)
+    (property "Reference" "Q?" (at 163.83 48.26 0)
       (effects (font (size 1.27 1.27)) (justify left))
     )
-    (property "Value" "BPC_IPP034N03L" (at 163.957 48.014 0)
+    (property "Value" "P03P4L-04" (at 163.83 45.72 0)
       (effects (font (size 1.27 1.27)) (justify left))
     )
-    (property "Footprint" "Package_TO_SOT_THT:TO-220-3_Vertical" (at 163.83 44.45 0)
+    (property "Footprint" "Package_TO_SOT_THT:TO-220-3_Vertical" (at 161.29 34.29 0)
       (effects (font (size 1.27 1.27)) hide)
     )
