File: cmd_tapis/cmd_tapis.kicad_sch (KiCad schematic)
At the start: 12 parts, among them X1 Trou, X2 Trou, X3 Trou, X4 Trou

Commit message: Modifs mineures: - Sérigraphie plus grosse - Commentaires sur schéma (consigne + D1 NM)
Parts:
- D?: value D -> 1N5818
Other:
- note added: "NM"
- note added: "Ne pas souder D2 côté relais mais sur le "dessus""
Changed lines of the file:
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@@
   (title_block
     (title "Commande tapis chauffant")
-    (date "2025-12-27")
-    (rev "Rev A")
+    (date "2026-01-19")
+    (rev "Rev B")
     (company "BPC")
     (comment 1 "Commande 12V/50mA - Sortie 230V / 10A")
@@
     (stroke (width 0) (type default))
   )
+  (rectangle (start 124.46 104.14) (end 137.16 127)
+    (stroke (width 0) (type dash))
+    (fill (type none))
+  )
+  (text_box "Rev:\n\n- D1 NM\n- Message avertissement D2\n- Aggrandissement sérigraphie\n"
+    (at 26.67 25.4 0) (size 43.18 15.24)
+    (stroke (width 0) (type default))
+    (fill (type none))
+    (effects (font (size 1.27 1.27)) (justify left top))
+  )
+  (text "NM" (at 128.27 119.38 0)
+    (effects (font (size 2.54 2.54) (thickness 0.508) bold) (justify left bottom))
+  )
+  (text "Ne pas souder D2 côté relais mais sur le \"dessus\"" (at 119.38 82.55 0)
+    (effects (font (size 1.27 1.27)) (justify left bottom))
+  )
   (symbol (lib_id "power:GND") (at 143.51 93.98 90) (unit 1)
     (in_bom yes) (on_board yes) (dnp no) (fields_autoplaced)
@@
     )
   )
-  (symbol (lib_id "bpc:BPC_TROU") (at 105.41 80.01 0) (unit 1)
-    (in_bom yes) (on_board yes) (dnp no) (fields_autoplaced)
-    (property "Reference" "X1" (at 106.045 78.986 0)
-      (effects (font (size 1.27 1.27)) (justify left))
-    )
-    (property "Value" "Trou" (at 106.045 81.034 0)
-      (effects (font (size 1.27 1.27)) (justify left))
-    )
-    (property "Footprint" "bpc:BPC_Trou4mm_Fixation" (at 105.41 77.47 0)
-      (effects (font (size 1.27 1.27)) hide)
-    )
-    (property "Datasheet" "" (at 105.41 80.01 0)
+  (symbol (lib_id "bpc:BPC_TROU") (at 121.92 148.59 0) (unit 1)
+    (in_bom yes) (on_board yes) (dnp no) (fields_autoplaced)
+    (property "Reference" "X1" (at 122.555 147.566 0)
+      (effects (font (size 1.27 1.27)) (justify left))
+    )
+    (property "Value" "Trou" (at 122.555 149.614 0)
+      (effects (font (size 1.27 1.27)) (justify left))
+    )
+    (property "Footprint" "bpc:BPC_Trou4mm_Fixation" (at 121.92 146.05 0)
+      (effects (font (size 1.27 1.27)) hide)
+    )
+    (property "Datasheet" "" (at 121.92 148.59 0)
       (effects (font (size 1.27 1.27)) hide)
     )
@@
       (effects (font (size 1.27 1.27)) (justify left))
     )
-    (property "Value" "D" (at 129.54 109.22 90)
+    (property "Value" "1N5818" (at 129.54 109.22 90)
       (effects (font (size 1.27 1.27)) (justify left))
     )
@@
     )
   )
-  (symbol (lib_id "bpc:BPC_TROU") (at 146.05 82.55 0) (unit 1)
-    (in_bom yes) (on_board yes) (dnp no) (fields_autoplaced)
-    (property "Reference" "X4" (at 146.685 81.526 0)
-      (effects (font (size 1.27 1.27)) (justify left))
-    )
-    (property "Value" "Trou" (at 146.685 83.574 0)
-      (effects (font (size 1.27 1.27)) (justify left))
-    )
-    (property "Footprint" "bpc:BPC_Trou4mm_Fixation" (at 146.05 80.01 0)
-      (effects (font (size 1.27 1.27)) hide)
-    )
-    (property "Datasheet" "" (at 146.05 82.55 0)
+  (symbol (lib_id "bpc:BPC_TROU") (at 162.56 151.13 0) (unit 1)
+    (in_bom yes) (on_board yes) (dnp no) (fields_autoplaced)
+    (property "Reference" "X4" (at 163.195 150.106 0)
+      (effects (font (size 1.27 1.27)) (justify left))
+    )
+    (property "Value" "Trou" (at 163.195 152.154 0)
+      (effects (font (size 1.27 1.27)) (justify left))
+    )
+    (property "Footprint" "bpc:BPC_Trou4mm_Fixation" (at 162.56 148.59 0)
+      (effects (font (size 1.27 1.27)) hide)
+    )
+    (property "Datasheet" "" (at 162.56 151.13 0)
       (effects (font (size 1.27 1.27)) hide)
     )
@@
     )
   )
-  (symbol (lib_id "bpc:BPC_TROU") (at 130.81 81.28 0) (unit 1)
-    (in_bom yes) (on_board yes) (dnp no) (fields_autoplaced)
-    (property "Reference" "X3" (at 131.445 80.256 0)
-      (effects (font (size 1.27 1.27)) (justify left))
-    )
-    (property "Value" "Trou" (at 131.445 82.304 0)
-      (effects (font (size 1.27 1.27)) (justify left))
-    )
-    (property "Footprint" "bpc:BPC_Trou4mm_Fixation" (at 130.81 78.74 0)
-      (effects (font (size 1.27 1.27)) hide)
-    )
-    (property "Datasheet" "" (at 130.81 81.28 0)
+  (symbol (lib_id "bpc:BPC_TROU") (at 147.32 149.86 0) (unit 1)
+    (in_bom yes) (on_board yes) (dnp no) (fields_autoplaced)
+    (property "Reference" "X3" (at 147.955 148.836 0)
+      (effects (font (size 1.27 1.27)) (justify left))
+    )
+    (property "Value" "Trou" (at 147.955 150.884 0)
+      (effects (font (size 1.27 1.27)) (justify left))
+    )
+    (property "Footprint" "bpc:BPC_Trou4mm_Fixation" (at 147.32 147.32 0)
+      (effects (font (size 1.27 1.27)) hide)
+    )
+    (property "Datasheet" "" (at 147.32 149.86 0)
       (effects (font (size 1.27 1.27)) hide)
     )
@@
     )
   )
-  (symbol (lib_id "bpc:BPC_TROU") (at 116.84 80.01 0) (unit 1)
-    (in_bom yes) (on_board yes) (dnp no) (fields_autoplaced)
-    (property "Reference" "X2" (at 117.475 78.986 0)
-      (effects (font (size 1.27 1.27)) (justify left))
-    )
-    (property "Value" "Trou" (at 117.475 81.034 0)
-      (effects (font (size 1.27 1.27)) (justify left))
-    )
-    (property "Footprint" "bpc:BPC_Trou4mm_Fixation" (at 116.84 77.47 0)
-      (effects (font (size 1.27 1.27)) hide)
-    )
-    (property "Datasheet" "" (at 116.84 80.01 0)
-      (effects (font (size 1.27 1.27)) hide)
-    )
+  (symbol (lib_id "bpc:BPC_TROU") (at 133.35 148.59 0) (unit 1)
+    (in_bom yes) (on_board yes) (dnp no) (fields_autoplaced)
+    (property "Reference" "X2" (at 133.985 147.566 0)
+      (effects (font (size 1.27 1.27)) (justify left))
+    )
+    (property "Value" "Trou" (at 133.985 149.614 0)
+      (effects (font (size 1.27 1.27)) (justify left))
+    )
+    (property "Footprint" "bpc:BPC_Trou4mm_Fixation" (at 133.35 146.05 0)
+      (effects (font (size 1.27 1.27)) hide)
+    )
+    (property "Datasheet" "" (at 133.35 148.59 0)
+      (effects (font (size 1.27 1.27)) hide)
+    )

Commit message: R=1k pour LED
Parts:
- R?: value R -> 1k
Changed lines of the file:
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@@
       (effects (font (size 1.27 1.27)))
     )
-    (property "Value" "R" (at 123.19 91.432 90)
+    (property "Value" "1k" (at 123.19 91.432 90)
       (effects (font (size 1.27 1.27)))
     )
@@
   )
   (symbol (lib_id "bpc:BPC_G2RL-1-DC12") (at 154.94 110.49 0) (unit 1)
-    (in_bom yes) (on_board yes) (dnp no) (fields_autoplaced)
-    (property "Reference" "RL1" (at 167.132 109.466 0)
+    (in_bom yes) (on_board yes) (dnp no)
+    (property "Reference" "RL1" (at 157.48 124.46 0)
       (effects (font (size 1.27 1.27)) (justify left))
     )
-    (property "Value" "BPC_G2RL-1-DC12" (at 167.132 111.514 0)
+    (property "Value" "BPC_G2RL-1-DC12" (at 151.13 127 0)
       (effects (font (size 1.27 1.27)) (justify left))
     )

Commit message: Améliorations:
- Isolation renforcée en coupant le PCB
- Ajout de passage pour colliers de serrage des cables
- Ajout diode en direct
- Ajout découplages
- Alignement grille 1mm
Parts:
- added C1: 20µF, Capacitor_THT:CP_Radial_D5.0mm_P2.50mm, symbol Device:C_Polarized
- added C2: 100nF, Capacitor_THT:C_Disc_D3.8mm_W2.6mm_P2.50mm, symbol Device:C
- added D?: 1N5818, Diode_THT:D_A-405_P10.16mm_Horizontal, symbol Device:D
Connections:
- net GND: now also C1.2, C2.2
- net at D?.1 (K), R?.1, RL1.1: now also C1.1, C2.1, D?.1 (K); no longer J?.1 (Pin_1)
- new net: D?.2 (A), J?.1 (Pin_1)
Other:
- note removed: "NM"
- moved on the sheet: D2, D?, J?, R?
